File: hardware/flounder-v2/flounder-v2.kicad_sch (KiCad schematic)
At the start: 11 parts, among them U1 Z8S180, U2 AS6C4008-55PCN, U3 SST39SF040, X1 18.432MHz

Commit message: Add PIO to v2
Parts:
- added C1, C2, C3, C4, C5: 0.1uF, Capacitor_THT:C_Disc_D5.0mm_W2.5mm_P5.00mm, symbol Device:C
- added C6, C7, C8, C9: 1uF, Capacitor_THT:CP_Radial_D5.0mm_P2.50mm, symbol Device:C_Polarized
- added J1: Conn_02x20_Odd_Even, Connector_PinHeader_2.54mm:PinHeader_2x20_P2.54mm_Vertical, symbol Connector_Generic:Conn_02x20_Odd_Even
- added J2: Conn_02x10_Odd_Even, Connector_PinHeader_2.54mm:PinHeader_2x10_P2.54mm_Vertical, symbol Connector_Generic:Conn_02x10_Odd_Even
- added J3, J4: DE9_Plug_MountingHoles, Connector_Dsub:DSUB-9_Male_Horizontal_P2.77x2.84mm_EdgePinOffset7.70mm_Housed_MountingHolesOffset9.12mm, symbol Connector:DE9_Plug_MountingHoles
- added R10, R8, R9: 4k7, Resistor_THT:R_Axial_DIN0207_L6.3mm_D2.5mm_P7.62mm_Horizontal, symbol Device:R
- added U4: MAX232, Package_DIP:DIP-16_W7.62mm_Socket, symbol Interface_UART:MAX232
- added U5: GAL16V8, Package_DIP:DIP-20_W7.62mm_Socket, symbol Logic_Programmable:GAL16V8
- added U6: Z84C20, Package_DIP:DIP-40_W15.24mm_Socket, symbol Interface:Z84C20
Connections:
- net +5V: now also C1.1, C2.1, C3.1, C4.1, C5.1, J1.1 (Pin_1), J1.2 (Pin_2), J2.1 (Pin_1), J2.2 (Pin_2), U4.16 (VCC), U5.20 (VCC), U6.26 (VCC)
- net A0: now also J1.13 (Pin_13), U6.6 (B/~{A})
- net A1: now also J1.14 (Pin_14), U6.5 (C/~{D})
- net A10: now also J1.25 (Pin_25)
- net A11: now also J1.26 (Pin_26)
- net A12: now also J1.27 (Pin_27)
- net A13: now also J1.28 (Pin_28), U5.1 (I1/CLK)
- net A14: now also J1.29 (Pin_29), U5.2 (I2)
- net A15: now also J1.30 (Pin_30), U5.3 (I3)
- net A16: now also J2.3 (Pin_3), U5.4 (I4)
- net A17: now also J2.4 (Pin_4), U5.5 (I5)
- net A18: now also J2.5 (Pin_5), U5.6 (I6)
- net A19: now also J2.6 (Pin_6), U5.7 (I7)
- net A2: now also J1.15 (Pin_15)
- net A3: now also J1.16 (Pin_16)
- net A4: now also J1.17 (Pin_17)
- net A5: now also J1.18 (Pin_18)
- net A6: now also J1.19 (Pin_19)
- net A7: now also J1.20 (Pin_20)
- net A8: now also J1.23 (Pin_23)
- net A9: now also J1.24 (Pin_24)
- net D0: now also J1.5 (Pin_5), U6.19 (D0)
- net D1: now also J1.6 (Pin_6), U6.20 (D1)
- net D2: now also J1.7 (Pin_7), U6.1 (D2)
- net D3: now also J1.8 (Pin_8), U6.40 (D3)
- net D4: now also J1.9 (Pin_9), U6.39 (D4)
- net D5: now also J1.10 (Pin_10), U6.38 (D5)
- net D6: now also J1.11 (Pin_11), U6.3 (D6)
- net D7: now also J1.12 (Pin_12), U6.2 (D7)
- net GND: now also U2.24 (OE#), U3.24 (OE), C1.2, C2.2, C3.2, C4.2, C5.2, J1.21 (Pin_21), J1.22 (Pin_22), J1.3 (Pin_3), J1.39 (Pin_39), J1.4 (Pin_4), J1.40 (Pin_40), J2.19 (Pin_19), J2.20 (Pin_20), R10.2, R8.2, R9.2, U4.15 (GND), U5.10 (GND), U6.11 (GND)
- net PHI: now also J1.35 (Pin_35), U6.25 (CLK)
- net /BUSACK: now also J2.8 (Pin_8)
- net /BUSREQ: now also J2.7 (Pin_7)
- net /INT0: now also J2.9 (Pin_9)
- net /INT1: now also J2.10 (Pin_10)
- net /INT2: now also J2.11 (Pin_11)
- net /IORQ: now also J1.34 (Pin_34), U5.9 (I9), U6.36 (~{IORQ})
- net /MREQ: now also J1.33 (Pin_33), U5.8 (I8)
- net /NMI: now also J2.12 (Pin_12)
- net /RD: now also J1.31 (Pin_31), U6.35 (~{RD})
- net /RESET: now also J1.37 (Pin_37), J1.38 (Pin_38)
- net /WAIT: now also J1.36 (Pin_36)
- net /WR: now also U2.29 (WE#), J1.32 (Pin_32)
- net /CTS0: now reaches U1.46 (/CTS0)
- net /CTS0: now also R10.1
- net /DCD0: now reaches U1.47 (/DCD0)
- net /DCD0: now also R9.1
- net /CTS1: now reaches U1.56 (RXS//CTS1)
- net /CTS1: now also R8.1
- net /ROM: now reaches U3.22 (CE)
- net /ROM: now also U5.13 (IO7)
- net /SRAM: now reaches U2.22 (CE#)
- net /SRAM: now also U5.12 (IO8)
- new net /PIO: U5.14 (IO6), U6.4 (~{CE})
Other:
- moved on the sheet: U2, U3
